File: Flight/OLD/FlightPCB.sch (EAGLE design)
At the start: 31 parts

Commit message: Fixes to Flight PCB
Fixed hole sizing/placement, BEC clearance, GPS clearance, terminal block clearance, resistor hole spacing. Minor silkscreen adjustments
Parts:
- R1, R2, R3, R4, R5, R6, R7: device rcl:R-US_0204/7 -> rcl:R-US_0204/5
