File: Flight/CALIPSO_V2-0/FlightPCB.sch (EAGLE design)
At the start: 65 parts, among them M1 MOSFET_60V_22A, M2 MOSFET_60V_22A, M3 MOSFET_60V_22A, M4 MOSFET_60V_22A, M5 MOSFET_60V_22A, M5V MOSFET_60V_22A, T4.1_L 24p, T4.1_R 24p

Commit message: Unsaved changes after 10/11/2020
changes that I made after 10/11/2020. I don't recall what all the changes are, but I will look soon.
Parts:
- LOGO1, LOGO2: value QWIIC_LOGO_4MM -> QWIIC_LOGO_CONNECTOR; device SparkFun-Aesthetics:QWIIC_LOGO_4MM -> SparkFun-Aesthetics:QWIIC_LOGO_CONNECTOR
Changed lines of the file:
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@@
 <part name="SUPPLY7" library="SparkFun-PowerSymbols" deviceset="VCC_2" device=""/>
 <part name="SUPPLY8" library="SparkFun-PowerSymbols" deviceset="VCC_2" device=""/>
-<part name="LOGO1" library="SparkFun-Aesthetics" deviceset="QWIIC_LOGO" device="_4MM"/>
-<part name="LOGO2" library="SparkFun-Aesthetics" deviceset="QWIIC_LOGO" device="_4MM"/>
+<part name="LOGO1" library="SparkFun-Aesthetics" deviceset="QWIIC_LOGO" device="_CONNECTOR" value="QWIIC_LOGO_CONNECTOR"/>
+<part name="LOGO2" library="SparkFun-Aesthetics" deviceset="QWIIC_LOGO" device="_CONNECTOR" value="QWIIC_LOGO_CONNECTOR"/>
 <part name="R14" library="SparkFun-Resistors" deviceset="1KOHM" device="-0603-1/10W-1%" value="1k"/>
 <part name="R15" library="SparkFun-Resistors" deviceset="20KOHM" device="-0603-1/10W-1%" value="20k"/>
